File: small-bipolar-supply.kicad_sch (KiCad schematic)
At the start: 16 parts, among them J1 USB_C_Receptacle_PowerOnly_6P, U1 LM2776

Commit message: chore: added connectors to schematic for castellated edges
Parts:
- added J10, J9: Conn_01x01, small-bipolar-supply:castellated_1_P2.54mm, symbol Connector_Generic:Conn_01x01
- added J2, J3, J4, J7, J8: Conn_01x02, small-bipolar-supply:castellated_2_P2.54mm, symbol Connector_Generic:Conn_01x02
- JP1: SILK (none) -> EN
Connections:
- net +5V: now also J7.1 (Pin_1), J7.2 (Pin_2)
- net -5V: now also J8.1 (Pin_1), J8.2 (Pin_2)
- net EN: now also J10.1 (Pin_1), J9.1 (Pin_1)
- net GND: now also J2.1 (Pin_1), J2.2 (Pin_2), J3.1 (Pin_1), J3.2 (Pin_2), J4.1 (Pin_1), J4.2 (Pin_2)
- net VOUT: now reaches C7.1, L2.1, U1.1 (VOUT)
Other:
- note added: "CASTELLATED CONNECTORS"
- title: Simple Bipolar Supply -> Small Bipolar Supply

Commit message: trace layout complete
Connections:
- net C+: now reaches C3.2, U1.5 (C1+)
- net C-: now reaches C3.1, U1.6 (C1-)
Changed lines of the file:
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@@
 	(wire
 		(pts
-			(xy 92.71 87.63) (xy 104.14 87.63)
+			(xy 92.71 87.63) (xy 101.6 87.63)
 		)
 		(stroke
@@
 	(wire
 		(pts
-			(xy 104.14 82.55) (xy 105.41 82.55)
+			(xy 101.6 82.55) (xy 105.41 82.55)
 		)
 		(stroke
@@
 	(wire
 		(pts
-			(xy 104.14 87.63) (xy 104.14 82.55)
+			(xy 101.6 87.63) (xy 101.6 82.55)
 		)
 		(stroke
@@
 		)
 	)
+	(label "C+"
+		(at 101.6 77.47 0)
+		(effects
+			(font
+				(size 1.27 1.27)
+				(thickness 0.1588)
+			)
+			(justify left bottom)
+		)
+	)
+	(label "C-"
+		(at 101.6 82.55 0)
+		(effects
+			(font
+				(size 1.27 1.27)
+				(thickness 0.1588)
+			)
+			(justify left bottom)
+		)
+	)

Commit message: Removed castellated edges & various layout tweaks
Parts:
- removed J10, J9: Conn_01x01, small-bipolar-supply:castellated_1_P2.54mm, symbol Connector_Generic:Conn_01x01
- removed J2, J3, J4, J7, J8: Conn_01x02, small-bipolar-supply:castellated_2_P2.54mm, symbol Connector_Generic:Conn_01x02
- removed JP1: SolderJumper_2_Open, Jumper:SolderJumper-2_P1.3mm_Open_RoundedPad1.0x1.5mm, symbol Jumper:SolderJumper_2_Open
- added U2: module_connectors, small-bipolar-supply:module-footprint, symbol simple-bipolar-supply:module_connectors
Connections:
- net EN is gone; now on net VBUS: U1.4 (EN)
- net +5V: now also U2.2 (+5V)
- net -5V: now also U2.3 (-5V)
- net GND: now also U2.1 (GND)
