File: electrical/simple-bipolar-suppy.kicad_sch (KiCad schematic)
At the start: 16 parts, among them J1 USB_C_Receptacle_PowerOnly_6P, U1 LM2776, U2 module_connectors

Commit message: various structure and documentation changes
Other:
- note added: "CONNECTORS"
- note removed: "CASTELLATED CONNECTORS"
- title: Small Bipolar Supply -> Simple Bipolar Supply
Changed lines of the file:
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@@
 	(paper "A5")
 	(title_block
-		(title "Small Bipolar Supply")
+		(title "Simple Bipolar Supply")
 		(date "2026-08-11")
 		(rev "B")
@@
 		)
 	)
-	(text "CASTELLATED CONNECTORS\n"
+	(text "CONNECTORS\n"
 		(exclude_from_sim no)
 		(at 41.148 76.962 0)
@@
 			(font
 				(size 1.27 1.27)
-				(thickness 0.254)
-				(bold yes)
+				(thickness 0.1588)
 			)
 			(justify right bottom)
@@
 		)
 		(instances
-			(project "small-bipolar-supply"
+			(project "simple-bipolar-suppy"
 				(path "/7769c9fd-d5c8-4d26-8add-365d4d4435ab"
 					(reference "C8")
@@
 		)
 		(instances
-			(project "small-bipolar-supply"
+			(project "simple-bipolar-suppy"
 				(path "/7769c9fd-d5c8-4d26-8add-365d4d4435ab"
 					(reference "C5")
@@
 		)
 		(instances
-			(project "small-bipolar-supply"
+			(project "simple-bipolar-suppy"
 				(path "/7769c9fd-d5c8-4d26-8add-365d4d4435ab"
 					(reference "R1")
@@
 		)
 		(instances
-			(project "small-bipolar-supply"
+			(project "simple-bipolar-suppy"
 				(path "/7769c9fd-d5c8-4d26-8add-365d4d4435ab"
 					(reference "#FLG03")
@@
 		)
 		(instances
-			(project "small-bipolar-supply"
+			(project "simple-bipolar-suppy"
 				(path "/7769c9fd-d5c8-4d26-8add-365d4d4435ab"
 					(reference "#FLG02")
@@
 		)
 		(instances
-			(project "small-bipolar-supply"
+			(project "simple-bipolar-suppy"
 				(path "/7769c9fd-d5c8-4d26-8add-365d4d4435ab"
 					(reference "C7")
@@
 		)
 		(instances
-			(project "small-bipolar-supply"
+			(project "simple-bipolar-suppy"
 				(path "/7769c9fd-d5c8-4d26-8add-365d4d4435ab"
 					(reference "#PWR03")
@@
 		)
 		(instances
-			(project "small-bipolar-supply"
+			(project "simple-bipolar-suppy"
 				(path "/7769c9fd-d5c8-4d26-8add-365d4d4435ab"
 					(reference "#PWR04")
@@
 		)
 		(instances
-			(project "small-bipolar-supply"
+			(project "simple-bipolar-suppy"
 				(path "/7769c9fd-d5c8-4d26-8add-365d4d4435ab"
 					(reference "C2")
@@
 		)
 		(instances
-			(project "small-bipolar-supply"
+			(project "simple-bipolar-suppy"
 				(path "/7769c9fd-d5c8-4d26-8add-365d4d4435ab"
 					(reference "#PWR010")
@@
 		)
 		(instances
-			(project "small-bipolar-supply"
+			(project "simple-bipolar-suppy"
 				(path "/7769c9fd-d5c8-4d26-8add-365d4d4435ab"
 					(reference "#PWR05")
@@
 		)
 		(instances
-			(project "small-bipolar-supply"
+			(project "simple-bipolar-suppy"
 				(path "/7769c9fd-d5c8-4d26-8add-365d4d4435ab"
 					(reference "L2")
@@
 		)
 		(instances
-			(project "small-bipolar-supply"
+			(project "simple-bipolar-suppy"
 				(path "/7769c9fd-d5c8-4d26-8add-365d4d4435ab"
 					(reference "#PWR06")
@@
 		)
 		(instances
-			(project "small-bipolar-supply"
+			(project "simple-bipolar-suppy"
 				(path "/7769c9fd-d5c8-4d26-8add-365d4d4435ab"
 					(reference "R2")
@@
 		)
 		(instances
-			(project "small-bipolar-supply"
+			(project "simple-bipolar-suppy"
 				(path "/7769c9fd-d5c8-4d26-8add-365d4d4435ab"
 					(reference "#FLG04")
@@
 		)
 		(instances
-			(project "small-bipolar-supply"
+			(project "simple-bipolar-suppy"
 				(path "/7769c9fd-d5c8-4d26-8add-365d4d4435ab"
 					(reference "U1")
@@
 		)
 		(instances
-			(project "small-bipolar-supply"
+			(project "simple-bipolar-suppy"
 				(path "/7769c9fd-d5c8-4d26-8add-365d4d4435ab"
 					(reference "#PWR08")
@@
 		)
 		(instances
-			(project "small-bipolar-supply"
+			(project "simple-bipolar-suppy"
 				(path "/7769c9fd-d5c8-4d26-8add-365d4d4435ab"
 					(reference "#PWR09")
@@
 		)
 		(instances
-			(project "small-bipolar-supply"
+			(project "simple-bipolar-suppy"
 				(path "/7769c9fd-d5c8-4d26-8add-365d4d4435ab"
 					(reference "C1")
@@
 		)
 		(instances
-			(project "small-bipolar-supply"
+			(project "simple-bipolar-suppy"
 				(path "/7769c9fd-d5c8-4d26-8add-365d4d4435ab"
 					(reference "L1")
@@
 		)
 		(instances
-			(project "small-bipolar-supply"
+			(project "simple-bipolar-suppy"
 				(path "/7769c9fd-d5c8-4d26-8add-365d4d4435ab"
 					(reference "#PWR014")
@@
 		)
 		(instances
-			(project "small-bipolar-supply"
+			(project "simple-bipolar-suppy"
 				(path "/7769c9fd-d5c8-4d26-8add-365d4d4435ab"
 					(reference "#PWR011")
@@
 		)
 		(instances
-			(project "small-bipolar-supply"
+			(project "simple-bipolar-suppy"
 				(path "/7769c9fd-d5c8-4d26-8add-365d4d4435ab"
 					(reference "#PWR07")
@@
 		)
 		(instances
-			(project "small-bipolar-supply"
+			(project "simple-bipolar-suppy"
 				(path "/7769c9fd-d5c8-4d26-8add-365d4d4435ab"
 					(reference "J1")
@@
 		)
 		(instances
-			(project "small-bipolar-supply"
+			(project "simple-bipolar-suppy"
 				(path "/7769c9fd-d5c8-4d26-8add-365d4d4435ab"
 					(reference "C9")
@@
 		)
 		(instances
-			(project "small-bipolar-supply"
+			(project "simple-bipolar-suppy"
 				(path "/7769c9fd-d5c8-4d26-8add-365d4d4435ab"
 					(reference "C6")
@@
 		)
 		(instances
-			(project "small-bipolar-supply"
+			(project "simple-bipolar-suppy"
 				(path "/7769c9fd-d5c8-4d26-8add-365d4d4435ab"
 					(reference "#FLG01")
@@
 		)
 		(instances
-			(project "small-bipolar-supply"
+			(project "simple-bipolar-suppy"
 				(path "/7769c9fd-d5c8-4d26-8add-365d4d4435ab"
 					(reference "U2")
@@
 		)
 		(instances
-			(project "small-bipolar-supply"
+			(project "simple-bipolar-suppy"
 				(path "/7769c9fd-d5c8-4d26-8add-365d4d4435ab"
 					(reference "C4")
@@
 		)
 		(instances
-			(project "small-bipolar-supply"
+			(project "simple-bipolar-suppy"
 				(path "/7769c9fd-d5c8-4d26-8add-365d4d4435ab"
 					(reference "C3")
@@
 		)
 		(instances
-			(project "small-bipolar-supply"
+			(project "simple-bipolar-suppy"
 				(path "/7769c9fd-d5c8-4d26-8add-365d4d4435ab"
 					(reference "#PWR01")
@@
 		)
 		(instances
-			(project "small-bipolar-supply"
+			(project "simple-bipolar-suppy"
 				(path "/7769c9fd-d5c8-4d26-8add-365d4d4435ab"
 					(reference "#PWR02")
@@
 		)
 		(instances
-			(project "small-bipolar-supply"
+			(project "simple-bipolar-suppy"
 				(path "/7769c9fd-d5c8-4d26-8add-365d4d4435ab"
 					(reference "#PWR012")
